Commit message: Update turtlebot3_fet.urdf.xacro

File: turtlebot3_description/urdf/turtlebot3_fet.urdf.xacro (robot description, xacro)
@@ -147,5 +147,5 @@
     <parent link="base_link"/>
     <child link="imu_link"/>
-    <origin xyz="0.12 -0.055 0.03" rpy="0 0 0"/>
+    <origin xyz="0.128 0.064 0.068" rpy="0 0 0"/>
   </joint>
   <link name="imu_link"/>
@@ -153,5 +153,5 @@
     <parent link="base_link"/>
     <child link="base_scan"/>
-    <origin xyz="0.12 0 0.135" rpy="0 0 0"/>
+    <origin xyz="0.10 0 0.18" rpy="0 0 0"/>
   </joint>
   <link name="base_scan">
